Commit message: Rolling update

File: models/buer.urdf (robot description, URDF)
Before this commit: robot buer, 16 links, 15 joints
Links:
- link head: geometry collision cylinder length=0.0004 radius=0.0004; visual mesh filename=stl/head.stl scale=0.0004 0.0004 0.0004
- link leg1_calf: geometry collision mesh filename=stl/calf.stl scale=0.0004 0.0004 0.0004; visual mesh filename=stl/calf.stl scale=0.0004 0.0004 0.0004
- link leg1_foot: geometry collision mesh filename=stl/foot.stl scale=0.0004 0.0004 0.0004; visual mesh filename=stl/foot.stl scale=0.0004 0.0004 0.0004
- link leg1_lap: geometry collision mesh filename=stl/lap.stl scale=0.0004 0.0004 0.0004; visual mesh filename=stl/lap.stl scale=0.0004 0.0004 0.0004
- link leg2_calf: geometry collision mesh filename=stl/calf.stl scale=0.0004 0.0004 0.0004; visual mesh filename=stl/calf.stl scale=0.0004 0.0004 0.0004
- link leg2_foot: geometry collision mesh filename=stl/foot.stl scale=0.0004 0.0004 0.0004; visual mesh filename=stl/foot.stl scale=0.0004 0.0004 0.0004
- link leg2_lap: geometry collision mesh filename=stl/lap.stl scale=0.0004 0.0004 0.0004; visual mesh filename=stl/lap.stl scale=0.0004 0.0004 0.0004
- link leg3_calf: geometry collision mesh filename=stl/calf.stl scale=0.0004 0.0004 0.0004; visual mesh filename=stl/calf.stl scale=0.0004 0.0004 0.0004
- link leg3_foot: geometry collision mesh filename=stl/foot.stl scale=0.0004 0.0004 0.0004; visual mesh filename=stl/foot.stl scale=0.0004 0.0004 0.0004
- link leg3_lap: geometry collision mesh filename=stl/lap.stl scale=0.0004 0.0004 0.0004; visual mesh filename=stl/lap.stl scale=0.0004 0.0004 0.0004
- link leg4_calf: geometry collision mesh filename=stl/calf.stl scale=0.0004 0.0004 0.0004; visual mesh filename=stl/calf.stl scale=0.0004 0.0004 0.0004
- link leg4_foot: geometry collision mesh filename=stl/foot.stl scale=0.0004 0.0004 0.0004; visual mesh filename=stl/foot.stl scale=0.0004 0.0004 0.0004
- link leg4_lap: geometry collision mesh filename=stl/lap.stl scale=0.0004 0.0004 0.0004; visual mesh filename=stl/lap.stl scale=0.0004 0.0004 0.0004
- link leg5_calf: geometry collision mesh filename=stl/calf.stl scale=0.0004 0.0004 0.0004; visual mesh filename=stl/calf.stl scale=0.0004 0.0004 0.0004
- link leg5_foot: geometry collision mesh filename=stl/foot.stl scale=0.0004 0.0004 0.0004; visual mesh filename=stl/foot.stl scale=0.0004 0.0004 0.0004
- link leg5_lap: geometry collision mesh filename=stl/lap.stl scale=0.0004 0.0004 0.0004; visual mesh filename=stl/lap.stl scale=0.0004 0.0004 0.0004
Joints:
- joint leg1_calf_joint: limit lower=-1.57 upper=1.57 effort=100.0 velocity=10.0 -> lower=-2.0 upper=2.0 effort=100.0 velocity=10.0; origin xyz=0 0 1 rpy=0 0 1.5708 -> xyz=0.0 0.0 0.4 rpy=0 0 1.5708
- joint leg1_foot_joint: limit lower=-1.57 upper=1.57 effort=100.0 velocity=10.0 -> lower=-2.0 upper=2.0 effort=100.0 velocity=10.0; origin xyz=0 0 0.8 rpy=0 0 0 -> xyz=0.0 0.0 0.32 rpy=0 0 0
- joint leg1_lap_joint: origin xyz=0 0.5505528 0 rpy=-1.57 0 0 -> xyz=0.0 0.22022112000000002 0.0 rpy=-1.57 0 0
- joint leg2_calf_joint: limit lower=-1.57 upper=1.57 effort=100.0 velocity=10.0 -> lower=-2.0 upper=2.0 effort=100.0 velocity=10.0; origin xyz=0 0 1 rpy=0 0 1.5708 -> xyz=0.0 0.0 0.4 rpy=0 0 1.5708
- joint leg2_foot_joint: limit lower=-1.57 upper=1.57 effort=100.0 velocity=10.0 -> lower=-2.0 upper=2.0 effort=100.0 velocity=10.0; origin xyz=0 0 0.8 rpy=0 0 0 -> xyz=0.0 0.0 0.32 rpy=0 0 0
- joint leg2_lap_joint: origin xyz=0.5236 0.1701 0.0 rpy=-1.57 0 -1.257 -> xyz=0.20944000000000002 0.06804 0.0 rpy=-1.57 0 -1.257
- joint leg3_calf_joint: limit lower=-1.57 upper=1.57 effort=100.0 velocity=10.0 -> lower=-2.0 upper=2.0 effort=100.0 velocity=10.0; origin xyz=0 0 1 rpy=0 0 1.5708 -> xyz=0.0 0.0 0.4 rpy=0 0 1.5708
- joint leg3_foot_joint: limit lower=-1.57 upper=1.57 effort=100.0 velocity=10.0 -> lower=-2.0 upper=2.0 effort=100.0 velocity=10.0; origin xyz=0 0 0.8 rpy=0 0 0 -> xyz=0.0 0.0 0.32 rpy=0 0 0
- joint leg3_lap_joint: origin xyz=0.3236 -0.4454 0.0 rpy=-1.57 0 -2.513 -> xyz=0.12944000000000003 -0.17816 0.0 rpy=-1.57 0 -2.513
- joint leg4_calf_joint: limit lower=-1.57 upper=1.57 effort=100.0 velocity=10.0 -> lower=-2.0 upper=2.0 effort=100.0 velocity=10.0; origin xyz=0 0 1 rpy=0 0 1.5708 -> xyz=0.0 0.0 0.4 rpy=0 0 1.5708
- joint leg4_foot_joint: limit lower=-1.57 upper=1.57 effort=100.0 velocity=10.0 -> lower=-2.0 upper=2.0 effort=100.0 velocity=10.0; origin xyz=0 0 0.8 rpy=0 0 0 -> xyz=0.0 0.0 0.32 rpy=0 0 0
- joint leg4_lap_joint: origin xyz=-0.3236 -0.4454 0.0 rpy=-1.57 0 2.513 -> xyz=-0.12944000000000003 -0.17816 0.0 rpy=-1.57 0 2.513
- joint leg5_calf_joint: limit lower=-1.57 upper=1.57 effort=100.0 velocity=10.0 -> lower=-2.0 upper=2.0 effort=100.0 velocity=10.0; origin xyz=0 0 1 rpy=0 0 1.5708 -> xyz=0.0 0.0 0.4 rpy=0 0 1.5708
- joint leg5_foot_joint: limit lower=-1.57 upper=1.57 effort=100.0 velocity=10.0 -> lower=-2.0 upper=2.0 effort=100.0 velocity=10.0; origin xyz=0 0 0.8 rpy=0 0 0 -> xyz=0.0 0.0 0.32 rpy=0 0 0
- joint leg5_lap_joint: origin xyz=-0.5236 0.1701 0.0 rpy=-1.57 0 1.257 -> xyz=-0.20944000000000002 0.06804 0.0 rpy=-1.57 0 1.257

File: models/buer.xacro (robot description, xacro)
@@ -66,5 +66,5 @@
       <origin xyz="${0*global_scale} ${0*global_scale} ${1000*global_scale}" rpy="0 0 ${calf_rpy}"/>
       <axis xyz="1 0 0"/>
-      <limit effort="100.0" velocity="10.0" lower="-1.57" upper="1.57"/>
+      <limit effort="100.0" velocity="10.0" lower="-2.0" upper="2.0"/>
     </joint>
     <!-- Foot link -->
@@ -75,5 +75,5 @@
       <origin xyz="${0*global_scale} ${0*global_scale} ${800*global_scale}" rpy="0 0 0"/>
       <axis xyz="1 0 0"/>
-      <limit effort="100.0" velocity="10.0" lower="-1.57" upper="1.57"/>
+      <limit effort="100.0" velocity="10.0" lower="-2.0" upper="2.0"/>
     </joint>
   </xacro:macro>
