Commit message: initial version

File: models/buer_fourlegs.urdf (robot description, URDF)
Before this commit: robot buer, 16 links, 15 joints
Links:
- removed link leg5_calf
- removed link leg5_foot
- removed link leg5_lap
Joints:
- removed joint leg5_calf_joint
- removed joint leg5_foot_joint
- removed joint leg5_lap_joint
- joint leg1_lap_joint: origin xyz=0.0 0.22022112000000002 0.0 rpy=-1.57 0 0 -> xyz=0.11 0.11 0.0 rpy=-1.57 0 0
- joint leg2_lap_joint: origin xyz=0.20944000000000002 0.06804 0.0 rpy=-1.57 0 -1.257 -> xyz=0.11 -0.11 0.0 rpy=-1.57 0 -1.5708
- joint leg3_lap_joint: origin xyz=0.12944000000000003 -0.17816 0.0 rpy=-1.57 0 -2.513 -> xyz=-0.11 -0.11 0.0 rpy=-1.57 0 3.1416
- joint leg4_lap_joint: origin xyz=-0.12944000000000003 -0.17816 0.0 rpy=-1.57 0 2.513 -> xyz=-0.11 0.11 0.0 rpy=-1.57 0 1.5708

File: models/buer_fourlegs.xacro (robot description, xacro)
@@ -79,8 +79,7 @@
   </xacro:macro>
   <!-- Instantiate legs -->
-  <xacro:leg idx="1" lx="0" ly="550.5528" lz="0" lroll="-1.57" lpitch="0" lyaw="0" calf_rpy="1.5708"/>
-  <xacro:leg idx="2" lx="523.6" ly="170.1" lz="0" lroll="-1.57" lpitch="0" lyaw="-1.257" calf_rpy="1.5708"/>
-  <xacro:leg idx="3" lx="323.6" ly="-445.4" lz="0" lroll="-1.57" lpitch="0" lyaw="-2.513" calf_rpy="1.5708"/>
-  <xacro:leg idx="4" lx="-323.6" ly="-445.4" lz="0" lroll="-1.57" lpitch="0" lyaw="2.513" calf_rpy="1.5708"/>
-  <xacro:leg idx="5" lx="-523.6" ly="170.1" lz="0" lroll="-1.57" lpitch="0" lyaw="1.257" calf_rpy="1.5708"/>
+<xacro:leg idx="1" lx="275" ly="275" lz="0" lroll="-1.57" lpitch="0" lyaw="0" calf_rpy="1.5708"/>
+<xacro:leg idx="2" lx="275" ly="-275" lz="0" lroll="-1.57" lpitch="0" lyaw="-1.5708" calf_rpy="1.5708"/>
+<xacro:leg idx="3" lx="-275" ly="-275" lz="0" lroll="-1.57" lpitch="0" lyaw="3.1416" calf_rpy="1.5708"/>
+<xacro:leg idx="4" lx="-275" ly="275" lz="0" lroll="-1.57" lpitch="0" lyaw="1.5708" calf_rpy="1.5708"/>
 </robot>

File: models/buer_stl.xacro (robot description, xacro)
@@ -79,8 +79,7 @@
   </xacro:macro>
   <!-- Instantiate legs -->
-  <xacro:leg idx="1" lx="0" ly="550.5528" lz="0" lroll="-1.57" lpitch="0" lyaw="0" calf_rpy="1.5708"/>
-  <xacro:leg idx="2" lx="523.6" ly="170.1" lz="0" lroll="-1.57" lpitch="0" lyaw="-1.257" calf_rpy="1.5708"/>
-  <xacro:leg idx="3" lx="323.6" ly="-445.4" lz="0" lroll="-1.57" lpitch="0" lyaw="-2.513" calf_rpy="1.5708"/>
-  <xacro:leg idx="4" lx="-323.6" ly="-445.4" lz="0" lroll="-1.57" lpitch="0" lyaw="2.513" calf_rpy="1.5708"/>
-  <xacro:leg idx="5" lx="-523.6" ly="170.1" lz="0" lroll="-1.57" lpitch="0" lyaw="1.257" calf_rpy="1.5708"/>
+<xacro:leg idx="1" lx="275" ly="275" lz="0" lroll="-1.57" lpitch="0" lyaw="0" calf_rpy="1.5708"/>
+<xacro:leg idx="2" lx="275" ly="-275" lz="0" lroll="-1.57" lpitch="0" lyaw="-1.5708" calf_rpy="1.5708"/>
+<xacro:leg idx="3" lx="-275" ly="-275" lz="0" lroll="-1.57" lpitch="0" lyaw="3.1416" calf_rpy="1.5708"/>
+<xacro:leg idx="4" lx="-275" ly="275" lz="0" lroll="-1.57" lpitch="0" lyaw="1.5708" calf_rpy="1.5708"/>
 </robot>

Commit message: Reward function refinement.

File: models/buer_fourlegs.urdf (robot description, URDF)
Before this commit: robot buer, 13 links, 12 joints
Joints:
- joint leg1_lap_joint: origin xyz=0.11 0.11 0.0 rpy=-1.57 0 0 -> xyz=0.0 0.11 0.0 rpy=-1.57 0 0
- joint leg2_lap_joint: origin xyz=0.11 -0.11 0.0 rpy=-1.57 0 -1.5708 -> xyz=0.11 0.0 0.0 rpy=-1.57 0 -1.5708
- joint leg3_lap_joint: origin xyz=-0.11 -0.11 0.0 rpy=-1.57 0 3.1416 -> xyz=0.0 -0.11 0.0 rpy=-1.57 0 3.1416
- joint leg4_lap_joint: origin xyz=-0.11 0.11 0.0 rpy=-1.57 0 1.5708 -> xyz=-0.11 0.0 0.0 rpy=-1.57 0 1.5708

File: models/buer_fourlegs.xacro (robot description, xacro)
@@ -79,7 +79,7 @@
   </xacro:macro>
   <!-- Instantiate legs -->
-<xacro:leg idx="1" lx="275" ly="275" lz="0" lroll="-1.57" lpitch="0" lyaw="0" calf_rpy="1.5708"/>
-<xacro:leg idx="2" lx="275" ly="-275" lz="0" lroll="-1.57" lpitch="0" lyaw="-1.5708" calf_rpy="1.5708"/>
-<xacro:leg idx="3" lx="-275" ly="-275" lz="0" lroll="-1.57" lpitch="0" lyaw="3.1416" calf_rpy="1.5708"/>
-<xacro:leg idx="4" lx="-275" ly="275" lz="0" lroll="-1.57" lpitch="0" lyaw="1.5708" calf_rpy="1.5708"/>
+<xacro:leg idx="1" lx="0" ly="275" lz="0" lroll="-1.57" lpitch="0" lyaw="0" calf_rpy="1.5708"/>
+<xacro:leg idx="2" lx="275" ly="0" lz="0" lroll="-1.57" lpitch="0" lyaw="-1.5708" calf_rpy="1.5708"/>
+<xacro:leg idx="3" lx="0" ly="-275" lz="0" lroll="-1.57" lpitch="0" lyaw="3.1416" calf_rpy="1.5708"/>
+<xacro:leg idx="4" lx="-275" ly="0" lz="0" lroll="-1.57" lpitch="0" lyaw="1.5708" calf_rpy="1.5708"/>
 </robot>
